File: pcb/controller/Power.sch (KiCad schematic (older format))
At the start: 34 parts, among them J2001 Conn_01x02_Female, U2001 LMZ14201, U2002 TPS82084, U2003 TPS735, U2004 TPS735

Commit message: updated schematic component values
Parts:
- C2001: value C -> 22n
- C2002: value C -> 10n
- C2003: value C -> 1u
- C2006: value CP1 -> 470u
- C2015: value CP2 -> 2200u
- FL2001: value EMI_Filter_CommonMode -> DLW5BTM501TQ2
- L2001: value L -> 1u
- R2001: value R -> 100k
- R2002: value R -> 34k
- R2003, R2004, R2007: value R -> 6.49k
- R2005: value R -> 41.2k
- R2008: value R -> 26.1k
- U2001: value LMZ14201 -> LMZ14201H
Changed lines of the file:
@@
 U 1 1 5C45A21F
 P 2500 2150
-F 0 "FL2001" H 2500 2428 50  0000 C CNN
-F 1 "EMI_Filter_CommonMode" H 2500 2337 50  0000 C CNN
+F 0 "FL2001" H 2700 2450 50  0000 C CNN
+F 1 "DLW5BTM501TQ2" H 2650 2350 50  0000 C CNN
 F 2 "wbraun_smd:DLW5BTM" V 2500 2190 50  0001 C CNN
 F 3 "~" V 2500 2190 50  0000 C CNN
@@
 P 3050 2200
 F 0 "C2003" H 3165 2246 50  0000 L CNN
-F 1 "C" H 3165 2155 50  0000 L CNN
+F 1 "1u" H 3165 2155 50  0000 L CNN
 F 2 "Capacitor_SMD:C_0805_2012Metric" H 3088 2050 50  0001 C CNN
 F 3 "~" H 3050 2200 50  0001 C CNN
@@
 P 3850 2200
 F 0 "C2006" H 3965 2246 50  0000 L CNN
-F 1 "CP1" H 3965 2155 50  0000 L CNN
+F 1 "470u" H 3965 2155 50  0000 L CNN
 F 2 "Capacitor_THT:CP_Radial_D10.0mm_P5.00mm" H 3850 2200 50  0001 C CNN
 F 3 "~" H 3850 2200 50  0001 C CNN
@@
 P 3450 1900
 F 0 "L2001" V 3640 1900 50  0000 C CNN
-F 1 "L" V 3549 1900 50  0000 C CNN
+F 1 "1u" V 3549 1900 50  0000 C CNN
 F 2 "Inductor_SMD:L_Vishay_IHLP-1212" H 3450 1900 50  0001 C CNN
 F 3 "~" H 3450 1900 50  0001 C CNN
@@
 P 2500 3950
 F 0 "U2001" H 2500 4515 50  0000 C CNN
-F 1 "LMZ14201" H 2500 4424 50  0000 C CNN
+F 1 "LMZ14201H" H 2500 4424 50  0000 C CNN
 F 2 "wbraun_smd:TO-PMOD-7" H 2100 3750 50  0001 C CNN
 F 3 "" H 2100 3750 50  0001 C CNN
@@
 P 1550 3850
 F 0 "C2002" V 1298 3850 50  0000 C CNN
-F 1 "C" V 1389 3850 50  0000 C CNN
+F 1 "10n" V 1389 3850 50  0000 C CNN
 F 2 "Capacitor_SMD:C_0402_1005Metric" H 1588 3700 50  0001 C CNN
 F 3 "~" H 1550 3850 50  0001 C CNN
@@
 P 1200 4550
 F 0 "C2001" H 1085 4504 50  0000 R CNN
-F 1 "C" H 1085 4595 50  0000 R CNN
+F 1 "22n" H 1085 4595 50  0000 R CNN
 F 2 "Capacitor_SMD:C_0402_1005Metric" H 1238 4400 50  0001 C CNN
 F 3 "~" H 1200 4550 50  0001 C CNN
@@
 P 1550 4550
 F 0 "R2002" H 1480 4504 50  0000 R CNN
-F 1 "R" H 1480 4595 50  0000 R CNN
+F 1 "34k" H 1480 4595 50  0000 R CNN
 F 2 "Resistor_SMD:R_0402_1005Metric" V 1480 4550 50  0001 C CNN
 F 3 "~" H 1550 4550 50  0001 C CNN
@@
 P 1900 4550
 F 0 "R2004" H 1970 4596 50  0000 L CNN
-F 1 "R" H 1970 4505 50  0000 L CNN
+F 1 "6.49k" H 1970 4505 50  0000 L CNN
 F 2 "Resistor_SMD:R_0402_1005Metric" V 1830 4550 50  0001 C CNN
 F 3 "~" H 1900 4550 50  0001 C CNN
@@
 P 2150 3250
 F 0 "R2005" V 1943 3250 50  0000 C CNN
-F 1 "R" V 2034 3250 50  0000 C CNN
+F 1 "41.2k" V 2034 3250 50  0000 C CNN
 F 2 "Resistor_SMD:R_0402_1005Metric" V 2080 3250 50  0001 C CNN
 F 3 "~" H 2150 3250 50  0001 C CNN
@@
 P 1650 3250
 F 0 "R2003" V 1443 3250 50  0000 C CNN
-F 1 "R" V 1534 3250 50  0000 C CNN
+F 1 "6.49k" V 1534 3250 50  0000 C CNN
 F 2 "Resistor_SMD:R_0402_1005Metric" V 1580 3250 50  0001 C CNN
 F 3 "~" H 1650 3250 50  0001 C CNN
@@
 P 750 4550
 F 0 "R2001" H 680 4504 50  0000 R CNN
-F 1 "R" H 680 4595 50  0000 R CNN
+F 1 "100k" H 680 4595 50  0000 R CNN
 F 2 "Resistor_SMD:R_0402_1005Metric" V 680 4550 50  0001 C CNN
 F 3 "~" H 750 4550 50  0001 C CNN
@@
 P 6800 5550
 F 0 "R2007" H 6730 5504 50  0000 R CNN
-F 1 "R" H 6730 5595 50  0000 R CNN
+F 1 "6.49k" H 6730 5595 50  0000 R CNN
 F 2 "Resistor_SMD:R_0402_1005Metric" V 6730 5550 50  0001 C CNN
 F 3 "~" H 6800 5550 50  0001 C CNN
@@
 P 6800 6000
 F 0 "R2008" H 6730 5954 50  0000 R CNN
-F 1 "R" H 6730 6045 50  0000 R CNN
+F 1 "26.1k" H 6730 6045 50  0000 R CNN
 F 2 "Resistor_SMD:R_0402_1005Metric" V 6730 6000 50  0001 C CNN
 F 3 "~" H 6800 6000 50  0001 C CNN
@@
 P 4350 2200
 F 0 "C2015" H 4465 2246 50  0000 L CNN
-F 1 "CP2" H 4465 2155 50  0000 L CNN
+F 1 "2200u" H 4465 2155 50  0000 L CNN
 F 2 "wbraun_smd:CAP_16mmx37mm_horizontal" H 4350 2200 50  0001 C CNN
 F 3 "~" H 4350 2200 50  0001 C CNN
